File: Clock/Clock.kicad_pcb (KiCad board)
At the start: 2 copper layers, 153 x 53 mm, 118 parts, among them J1 PWR, Q1 SI2308, U1 ATmega328P-A, U2 DS1307Z+, U4 AT24CS32, Y1 16Mhz, Y2 32.768Khz

Commit message: update
Parts:
- removed BT1: CR2032, Battery:BatteryHolder_Keystone_1060_1x2032
- removed BZ1: Buzzer, Buzzer_Beeper:Buzzer_1206
- removed C1, C3, C6, C7, C8: 100nF, Capacitor_SMD:C_0805_2012Metric_Pad1.18x1.45mm_HandSolder
- removed C2, C4: 22pF, Capacitor_SMD:C_0805_2012Metric_Pad1.18x1.45mm_HandSolder
- removed C5: 10uF, Capacitor_Tantalum_SMD:CP_EIA-3216-10_Kemet-I_Pad1.58x1.35mm_HandSolder
- removed D1: LED, LED_SMD:LED_0805_2012Metric_Pad1.15x1.40mm_HandSolder
- removed D2, D3: 1N4007, Diode_SMD:D_SMA
- removed DHT1: Conn_01x03, Connector_PinSocket_2.54mm:PinSocket_1x03_P2.54mm_Vertical
- removed FTDI1: Conn_01x05, Connector_PinHeader_2.54mm:PinHeader_1x05_P2.54mm_Vertical
- removed J1: PWR, Connector_PinSocket_2.54mm:PinSocket_1x02_P2.54mm_Vertical
- removed Q1: SI2308, Package_TO_SOT_SMD:SOT-23
- removed R1: 1K, Resistor_SMD:R_0805_2012Metric_Pad1.20x1.40mm_HandSolder
- removed R2: 10K, Resistor_SMD:R_0805_2012Metric_Pad1.20x1.40mm_HandSolder
- removed R5: 100, Resistor_SMD:R_0805_2012Metric_Pad1.20x1.40mm_HandSolder
- removed R6: 365, Resistor_SMD:R_0805_2012Metric_Pad1.20x1.40mm_HandSolder
- removed R7: 1.5M, Resistor_SMD:R_0805_2012Metric_Pad1.20x1.40mm_HandSolder
- removed R8: 510K, Resistor_SMD:R_0805_2012Metric_Pad1.20x1.40mm_HandSolder
- removed R9: 200, Resistor_SMD:R_0805_2012Metric_Pad1.20x1.40mm_HandSolder
- removed U1: ATmega328P-A, Package_QFP:TQFP-32_7x7mm_P0.8mm
- removed U2: DS1307Z+, Package_SO:SOIC-8_3.9x4.9mm_P1.27mm
- removed U4: AT24CS32, Package_SO:SOIC-8_3.9x4.9mm_P1.27mm
- removed Y1: 16Mhz, Crystal:Crystal_SMD_3225-4Pin_3.2x2.5mm_HandSoldering
- removed Y2: 32.768Khz, Crystal:Crystal_SMD_SeikoEpson_MC306-4Pin_8.0x3.2mm_HandSoldering
- removed reset: SW_Push, Button_Switch_SMD:SW_SPST_SKQG_WithStem
Routing:
- net +5V: track 888.6 -> 0.00 mm, vias 15 -> 0
- net ControlLed: track 136.0 -> 0.00 mm, vias 1 -> 0
- net connect_1: track 62.3 -> 0.00 mm
- net connect_5: track 53.6 -> 0.00 mm, vias 2 -> 0
- net connect_4: track 51.0 -> 0.00 mm
- net connect_6: track 43.8 -> 0.00 mm
- net connect_3: track 41.6 -> 0.00 mm
- net SDA: track 35.4 -> 0.00 mm, vias 2 -> 0
- net Net-(D36-Pad2): track 35.2 -> 0.00 mm
- net SCL: track 34.7 -> 0.00 mm, vias 2 -> 0
- net connect_7: track 34.3 -> 0.00 mm
- net BT_SETUP: track 28.8 -> 0.00 mm, vias 3 -> 0
- net BT_DOWN: track 28.1 -> 0.00 mm, vias 1 -> 0
- net Net-(D11-Pad2): track 26.5 -> 0.00 mm
- net Net-(D28-Pad2): track 25.0 -> 0.00 mm
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- removed copper zone on B.Cu, net GND
- removed copper zone on F.Cu, net GND
- removed copper zone on B.Cu, net Net-(BT1-Pad1)
- removed copper zone on B.Cu, net Net-(D3-Pad2)
- removed copper zone on B.Cu, net OSC1
- removed copper zone on B.Cu, net OSC2
- removed copper zone on B.Cu, net Reset
Other:
- board text removed: "CLOCK LED"
- board text removed: "DATA"
- board text removed: "DTR"
- board text removed: "GND"
- board text removed: "RX"
- board text removed: "TX"
- board text removed: "made by V.C.H"
