File: Clock/Clock.kicad_sch (KiCad schematic)
At the start: 26 parts

Commit message: update PCB 09/1/2022
Parts:
- removed Y?: 32.768Khz, Crystal:Crystal_C26-LF_D2.1mm_L6.5mm_Horizontal, symbol Device:Crystal
- added AL1, AL2, DOWN1, SET1, UP1: SW_Push, Button_Switch_SMD:SW_Push_1P1T-3x6, symbol Switch:SW_Push
- added BZ1: Buzzer, Buzzer_Beeper:Buzzer_1206, symbol Device:Buzzer
- added C10, C11, C12, C13, C14: 100nF, Capacitor_SMD:C_0805_2012Metric_Pad1.18x1.45mm_HandSolder, symbol Device:C_Small
- added D2: 1N4007, Diode_SMD:D_SMA, symbol Diode:1N4007
- added DHT1: Conn_01x03, Connector_PinSocket_2.54mm:PinSocket_1x03_P2.54mm_Vertical, symbol Connector_Generic:Conn_01x03
- added J1: PWR, Connector_PinSocket_2.54mm:PinSocket_1x02_P2.54mm_Vertical, symbol Connector_Generic:Conn_01x02
- added Q1: SI2308, Package_TO_SOT_SMD:SOT-23, symbol Device:Q_NMOS_GSD
- added R11, R12, R13, R14, R15, R5: 100, Resistor_SMD:R_0805_2012Metric_Pad1.20x1.40mm_HandSolder, symbol Device:R_Small_US
- added Y2: 32.768Khz, Crystal:Crystal_SMD_SeikoEpson_MC306-4Pin_8.0x3.2mm_HandSoldering, symbol Device:Crystal_GND23
- C6: renamed from C?; footprint (none) -> Capacitor_SMD:C_0805_2012Metric_Pad1.18x1.45mm_HandSolder
- reset1: renamed from reset; footprint (none) -> Button_Switch_SMD:SW_SPST_SKQG_WithStem
- gave numbers to parts that had none: 22
- renumbered FTDI to FTDI1
Connections:
- net +5V: now also FTDI1.1 (Pin_1), BZ1.1 (-), D2.1 (K), DHT1.1 (Pin_1), J1.2 (Pin_2), R11.2, R12.2, R13.2, R14.2, R15.2; no longer FTDI1.4 (Pin_4)
- net ControlLed: now also U1.9 (PD5); no longer U1.1 (PD3)
- net DTR: now also FTDI1.4 (Pin_4); no longer FTDI1.1 (Pin_1)
- net GND: now also AL1.2, AL2.2, C10.1, C11.1, C12.1, C13.1, C14.1, DHT1.3 (Pin_3), DOWN1.2, J1.1 (Pin_1), Q1.2 (S), SET1.2, UP1.2
- net at U2.1 (X1): now also Y2.4
- net at R6.1, U2.2 (X2): now also Y2.1
- net DHT: now reaches U1.10 (PD6)
- net DHT: now also DHT1.2 (Pin_2)
- net Alarm: now reaches U1.11 (PD7)
- net Alarm: now also R5.1
- net BT_DOWN: now reaches U1.2 (PD4)
- net BT_DOWN: now also C14.2, DOWN1.1, R15.1
- net BT_SETUP: now reaches U1.32 (PD2)
- net BT_SETUP: now also C11.2, R12.1, SET1.1
- new net: Q1.1 (G), R5.2
- new net: BZ1.2 (+), D2.2 (A), Q1.3 (D)
- new net BT_ALARM1: AL1.1, C10.2, R11.1
- new net BT_ALARM2: AL2.1, C12.2, R13.1
- new net BT_UP: C13.2, R14.1, U1.1 (PD3), UP1.1
Other:
- note added: "ALARM"
- note added: "BUTTON"
- note added: "DHT11"
- moved on the sheet: R6

Commit message: update
Parts:
- removed BT1: CR2032, Battery:BatteryHolder_Keystone_1060_1x2032, symbol Device:Battery_Cell
- removed BZ1: Buzzer, Buzzer_Beeper:Buzzer_1206, symbol Device:Buzzer
- removed C1, C3, C6, C7, C8: 100nF, Capacitor_SMD:C_0805_2012Metric_Pad1.18x1.45mm_HandSolder, symbol Device:C_Small
- removed C2, C4: 22pF, Capacitor_SMD:C_0805_2012Metric_Pad1.18x1.45mm_HandSolder, symbol Device:C_Small
- removed C5: 10uF, Capacitor_Tantalum_SMD:CP_EIA-3216-10_Kemet-I_Pad1.58x1.35mm_HandSolder, symbol Device:C_Polarized_Small
- removed D1: LED, LED_SMD:LED_0805_2012Metric_Pad1.15x1.40mm_HandSolder, symbol Device:LED
- removed D2, D3: 1N4007, Diode_SMD:D_SMA, symbol Diode:1N4007
- removed DHT1: Conn_01x03, Connector_PinSocket_2.54mm:PinSocket_1x03_P2.54mm_Vertical, symbol Connector_Generic:Conn_01x03
- removed FTDI1: Conn_01x05, Connector_PinHeader_2.54mm:PinHeader_1x05_P2.54mm_Vertical, symbol Connector_Generic:Conn_01x05
- removed J1: PWR, Connector_PinSocket_2.54mm:PinSocket_1x02_P2.54mm_Vertical, symbol Connector_Generic:Conn_01x02
- removed Q1: SI2308, Package_TO_SOT_SMD:SOT-23, symbol Device:Q_NMOS_GSD
- removed R1: 1K, Resistor_SMD:R_0805_2012Metric_Pad1.20x1.40mm_HandSolder, symbol Device:R_Small_US
- removed R2, R3, R4: 10K, Resistor_SMD:R_0805_2012Metric_Pad1.20x1.40mm_HandSolder, symbol Device:R_Small_US
- removed R5: 100, Resistor_SMD:R_0805_2012Metric_Pad1.20x1.40mm_HandSolder, symbol Device:R_Small_US
- removed R6: 365, Resistor_SMD:R_0805_2012Metric_Pad1.20x1.40mm_HandSolder, symbol Device:R_Small_US
- removed R7: 1.5M, Resistor_SMD:R_0805_2012Metric_Pad1.20x1.40mm_HandSolder, symbol Device:R_Small_US
- removed R8: 510K, Resistor_SMD:R_0805_2012Metric_Pad1.20x1.40mm_HandSolder, symbol Device:R_Small_US
- removed R9: 200, Resistor_SMD:R_0805_2012Metric_Pad1.20x1.40mm_HandSolder, symbol Device:R_Small_US
- removed U1: ATmega328P-A, Package_QFP:TQFP-32_7x7mm_P0.8mm, symbol MCU_Microchip_ATmega:ATmega328P-A
- removed U2: DS1307Z+, Package_SO:SOIC-8_3.9x4.9mm_P1.27mm, symbol Timer_RTC:DS1307Z+
- removed U4: AT24CS32, Package_SO:SOIC-8_3.9x4.9mm_P1.27mm, symbol Memory_EEPROM:AT24CS32-SSHM
- removed Y1: 16Mhz, Crystal:Crystal_SMD_3225-4Pin_3.2x2.5mm_HandSoldering, symbol Device:Crystal_GND24
- removed Y2: 32.768Khz, Crystal:Crystal_SMD_SeikoEpson_MC306-4Pin_8.0x3.2mm_HandSoldering, symbol Device:Crystal_GND23
- removed reset1: SW_Push, Button_Switch_SMD:SW_SPST_SKQG_WithStem, symbol Switch:SW_Push
Other:
- note removed: "ALARM"
- note removed: "BUTTON"
- note removed: "DHT11"
- note removed: "RTC"
- moved on the sheet: AL1, AL2, C10, C11, C12, C13, C14, DOWN1, R11, R12, R13, R14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
